File: pcb/usb-fanctl.brd (EAGLE design)
At the start: 50 x 50 mm, 68 parts, among them CON1 KF301-2P, CON2 KF301-2P, CON3 KF301-2P, CON4 KF301-2P, CON5 KF301-2P, CON6 KF301-2P, CON7 KF301-2P, CON8 KF301-2P, Q1 AO3400, Q2 AO3400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

Commit message: Add production files
Signed-off-by: João Silva <jgc3silva@gmail.com>
Parts:
- added C15, C16: 22uF, Capacitor:CAP1206
Connections:
- net GND: now also C15.2, C16.2
- net VEXT: now also C15.1, C16.1
Routing:
- net VEXT: vias 26 -> 32
Changed lines of the file:
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@@
 <drawing>
 <settings>
-<setting alwaysvectorfont="no"/>
+<setting alwaysvectorfont="yes"/>
 <setting verticaltext="up"/>
 </settings>
-<grid distance="0.1" unitdist="mm" unit="mm" style="lines" multiple="1" display="yes" altdistance="0.05" altunitdist="mm" altunit="mm"/>
+<grid distance="0.25" unitdist="mm" unit="mm" style="lines" multiple="1" display="yes" altdistance="0.05" altunitdist="mm" altunit="mm"/>
 <layers>
 <layer number="1" name="Top" color="4" fill="1" visible="yes" active="yes"/>
@@
 <attribute name="VOLTAGE" value="" x="29.5" y="21.5" size="0.8" layer="27" font="vector" ratio="10" rot="R270" display="off"/>
 </element>
+<element name="C15" library="Capacitor" package="CAP1206" value="22uF" x="44" y="8" smashed="yes">
+<attribute name="NAME" x="43.25" y="6.5" size="0.8" layer="25" font="vector" ratio="10" rot="SR0" align="center-left"/>
+<attribute name="VOLTAGE" value="" x="44" y="8" size="1.778" layer="27" display="off"/>
+</element>
+<element name="C16" library="Capacitor" package="CAP1206" value="22uF" x="44" y="42" smashed="yes">
+<attribute name="NAME" x="43.25" y="43.5" size="0.8" layer="25" font="vector" ratio="10" rot="SR0" align="center-left"/>
+<attribute name="VOLTAGE" value="" x="44" y="42.1" size="1.778" layer="27" display="off"/>
+</element>
 </elements>
 <signals>
@@
 <via x="28.1" y="31.9" extent="1-16" drill="0.2"/>
 <via x="18.5" y="12.2" extent="1-16" drill="0.2"/>
+<contactref element="C15" pad="2"/>
+<contactref element="C16" pad="2"/>
+<via x="46.75" y="8.75" extent="1-16" drill="0.3"/>
+<via x="46.75" y="8" extent="1-16" drill="0.3"/>
+<via x="46.75" y="7.25" extent="1-16" drill="0.3"/>
+<via x="46.75" y="42.75" extent="1-16" drill="0.3"/>
+<via x="46.75" y="42" extent="1-16" drill="0.3"/>
+<via x="46.75" y="41.25" extent="1-16" drill="0.3"/>
 </signal>
 <signal name="N$1">
@@
 <wire x1="26.75" y1="14" x2="26.75" y2="11.278" width="0.254" layer="1"/>
 <wire x1="26.75" y1="11.278" x2="26.472" y2="11" width="0.254" layer="1"/>
+<contactref element="C15" pad="1"/>
+<contactref element="C16" pad="1"/>
+<polygon width="0.2" layer="1" thermals="no">
+<vertex x="43" y="41"/>
+<vertex x="41" y="41"/>
+<vertex x="41" y="43"/>
+<vertex x="43" y="43"/>
+</polygon>
+<via x="41.25" y="42.75" extent="1-16" drill="0.3"/>
+<via x="41.25" y="42" extent="1-16" drill="0.3"/>
+<via x="41.25" y="41.25" extent="1-16" drill="0.3"/>
+<polygon width="0.2" layer="1" thermals="no">
+<vertex x="43" y="7"/>
+<vertex x="41" y="7"/>
+<vertex x="41" y="9"/>
+<vertex x="43" y="9"/>
+</polygon>
+<via x="41.25" y="8.75" extent="1-16" drill="0.3"/>
+<via x="41.25" y="8" extent="1-16" drill="0.3"/>
+<via x="41.25" y="7.25" extent="1-16" drill="0.3"/>
 </signal>
 <signal name="PWM0">
@@
 </signals>
 <mfgpreviewcolors>
-<mfgpreviewcolor name="soldermaskcolor" color="0xC8008000"/>
+<mfgpreviewcolor name="soldermaskcolor" color="0xC83C0480"/>
 <mfgpreviewcolor name="silkscreencolor" color="0xFFFEFEFE"/>
 <mfgpreviewcolor name="backgroundcolor" color="0xFF282828"/>
-<mfgpreviewcolor name="coppercolor" color="0xFFFFBF00"/>
+<mfgpreviewcolor name="coppercolor" color="0xFFC1C1C1"/>
 <mfgpreviewcolor name="substratecolor" color="0xFF786E46"/>
 </mfgpreviewcolors>
