File: pcb/usb-fanctl.sch (EAGLE design)
At the start: 68 parts, among them CON1 KF301-2P, CON2 KF301-2P, CON3 KF301-2P, CON4 KF301-2P, CON5 KF301-2P, CON6 KF301-2P, CON7 KF301-2P, CON8 KF301-2P, Q1 AO3400, Q2 AO3400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

Commit message: Add production files
Signed-off-by: João Silva <jgc3silva@gmail.com>
Parts:
- added C15, C16: 22uF, Capacitor:CAPACITOR-1206
Connections:
- net GND: now also C15.C2, C16.C2
- net VEXT: now also C15.C1, C16.C1
Changed lines of the file:
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@@
 <part name="GND38" library="Supply Symbol" deviceset="GND" device=""/>
 <part name="VIN9" library="Supply Symbol" deviceset="VEXT" device=""/>
+<part name="C15" library="Capacitor" deviceset="CAPACITOR" device="-1206" value="22uF"/>
+<part name="VIN10" library="Supply Symbol" deviceset="VEXT" device=""/>
+<part name="GND39" library="Supply Symbol" deviceset="GND" device=""/>
+<part name="C16" library="Capacitor" deviceset="CAPACITOR" device="-1206" value="22uF"/>
+<part name="VIN11" library="Supply Symbol" deviceset="VEXT" device=""/>
+<part name="GND40" library="Supply Symbol" deviceset="GND" device=""/>
 </parts>
 <sheets>
@@
 <attribute name="VALUE" x="332.74" y="66.04" size="1.778" layer="96" rot="R90"/>
 </instance>
+<instance part="C15" gate="G$1" x="467.36" y="157.48" smashed="yes" rot="R270">
+<attribute name="VALUE" x="464.5914" y="157.48" size="1.778" layer="96" ratio="10" rot="SR270" align="top-left"/>
+<attribute name="NAME" x="470.1286" y="157.48" size="1.778" layer="95" ratio="10" rot="SR270"/>
+<attribute name="VOLTAGE" x="462.0514" y="157.48" size="1.778" layer="97" ratio="10" rot="SR270" align="top-left"/>
+</instance>
+<instance part="VIN10" gate="G$1" x="467.36" y="162.56" smashed="yes">
+<attribute name="VALUE" x="464.82" y="160.02" size="1.778" layer="96" rot="R90"/>
+</instance>
+<instance part="GND39" gate="G$1" x="467.36" y="144.78" smashed="yes">
+<attribute name="VALUE" x="467.36" y="139.7" size="1.778" layer="96" align="bottom-center"/>
+</instance>
+<instance part="C16" gate="G$1" x="480.06" y="157.48" smashed="yes" rot="R270">
+<attribute name="VALUE" x="477.2914" y="157.48" size="1.778" layer="96" ratio="10" rot="SR270" align="top-left"/>
+<attribute name="NAME" x="482.8286" y="157.48" size="1.778" layer="95" ratio="10" rot="SR270"/>
+<attribute name="VOLTAGE" x="474.7514" y="157.48" size="1.778" layer="97" ratio="10" rot="SR270" align="top-left"/>
+</instance>
+<instance part="VIN11" gate="G$1" x="480.06" y="162.56" smashed="yes">
+<attribute name="VALUE" x="477.52" y="160.02" size="1.778" layer="96" rot="R90"/>
+</instance>
+<instance part="GND40" gate="G$1" x="480.06" y="144.78" smashed="yes">
+<attribute name="VALUE" x="480.06" y="139.7" size="1.778" layer="96" align="bottom-center"/>
+</instance>
 </instances>
 <busses>
@@
 <pinref part="C14" gate="G$1" pin="C2"/>
 </segment>
+<segment>
+<pinref part="GND39" gate="G$1" pin="GND"/>
+<wire x1="467.36" y1="149.86" x2="467.36" y2="144.78" width="0.1524" layer="91"/>
+<pinref part="C15" gate="G$1" pin="C2"/>
+</segment>
+<segment>
+<pinref part="GND40" gate="G$1" pin="GND"/>
+<wire x1="480.06" y1="149.86" x2="480.06" y2="144.78" width="0.1524" layer="91"/>
+<pinref part="C16" gate="G$1" pin="C2"/>
+</segment>
 </net>
 <net name="N$1" class="0">
@@
 <pinref part="VIN9" gate="G$1" pin="VEXT"/>
 </segment>
+<segment>
+<pinref part="VIN10" gate="G$1" pin="VEXT"/>
+<wire x1="467.36" y1="157.48" x2="467.36" y2="162.56" width="0.1524" layer="91"/>
+<pinref part="C15" gate="G$1" pin="C1"/>
+</segment>
+<segment>
+<pinref part="VIN11" gate="G$1" pin="VEXT"/>
+<wire x1="480.06" y1="157.48" x2="480.06" y2="162.56" width="0.1524" layer="91"/>
+<pinref part="C16" gate="G$1" pin="C1"/>
+</segment>
 </net>
